File: ARM.sch (KiCad schematic (older format))
At the start: 21 parts

Commit message: Adding IR Sensor
Parts:
- gave numbers to parts that had none: 21
Changed lines of the file:
@@
 $EndDescr
 $Comp
-L +3V3 #PWR?
+L +3V3 #PWR019
 U 1 1 5A9B46CA
 P 2350 2500
-F 0 "#PWR?" H 2350 2350 50  0001 C CNN
+F 0 "#PWR019" H 2350 2350 50  0001 C CNN
 F 1 "+3V3" H 2350 2640 50  0000 C CNN
 F 2 "" H 2350 2500 50  0001 C CNN
@@
 $EndComp
 $Comp
-L C C?
+L C C11
 U 1 1 5A9B46E6
 P 1950 3350
-F 0 "C?" H 1975 3450 50  0000 L CNN
+F 0 "C11" H 1975 3450 50  0000 L CNN
 F 1 "10nF" H 1975 3250 50  0000 L CNN
 F 2 "" H 1988 3200 50  0001 C CNN
@@
 $EndComp
 $Comp
-L C C?
+L C C10
 U 1 1 5A9B4725
 P 1800 4850
-F 0 "C?" H 1825 4950 50  0000 L CNN
+F 0 "C10" H 1825 4950 50  0000 L CNN
 F 1 "100nF" H 1825 4750 50  0000 L CNN
 F 2 "" H 1838 4700 50  0001 C CNN
@@
 $EndComp
 $Comp
-L C C?
+L C C12
 U 1 1 5A9B475A
 P 6500 2450
-F 0 "C?" H 6525 2550 50  0000 L CNN
+F 0 "C12" H 6525 2550 50  0000 L CNN
 F 1 "100nF" H 6525 2350 50  0000 L CNN
 F 2 "" H 6538 2300 50  0001 C CNN
@@
 $EndComp
 $Comp
-L C C?
+L C C13
 U 1 1 5A9B479A
 P 6650 3750
-F 0 "C?" H 6675 3850 50  0000 L CNN
+F 0 "C13" H 6675 3850 50  0000 L CNN
 F 1 "100nF" H 6675 3650 50  0000 L CNN
 F 2 "" H 6688 3600 50  0001 C CNN
@@
 $EndComp
 $Comp
-L +3V3 #PWR?
+L +3V3 #PWR020
 U 1 1 5A9B480C
 P 1700 3500
-F 0 "#PWR?" H 1700 3350 50  0001 C CNN
+F 0 "#PWR020" H 1700 3350 50  0001 C CNN
 F 1 "+3V3" H 1700 3640 50  0000 C CNN
 F 2 "" H 1700 3500 50  0001 C CNN
@@
 $EndComp
 $Comp
-L GND #PWR?
+L GND #PWR021
 U 1 1 5A9B4836
 P 1500 3200
-F 0 "#PWR?" H 1500 2950 50  0001 C CNN
+F 0 "#PWR021" H 1500 2950 50  0001 C CNN
 F 1 "GND" H 1500 3050 50  0000 C CNN
 F 2 "" H 1500 3200 50  0001 C CNN
@@
 	2150 3500 1700 3500
 $Comp
-L +3V3 #PWR?
+L +3V3 #PWR022
 U 1 1 5A9B48AF
 P 1550 5000
-F 0 "#PWR?" H 1550 4850 50  0001 C CNN
+F 0 "#PWR022" H 1550 4850 50  0001 C CNN
 F 1 "+3V3" H 1550 5140 50  0000 C CNN
 F 2 "" H 1550 5000 50  0001 C CNN
@@
 $EndComp
 $Comp
-L GND #PWR?
+L GND #PWR023
 U 1 1 5A9B48B5
 P 1350 4700
-F 0 "#PWR?" H 1350 4450 50  0001 C CNN
+F 0 "#PWR023" H 1350 4450 50  0001 C CNN
 F 1 "GND" H 1350 4550 50  0000 C CNN
 F 2 "" H 1350 4700 50  0001 C CNN
@@
 Connection ~ 1800 4700
 $Comp
-L +3V3 #PWR?
+L +3V3 #PWR024
 U 1 1 5A9B4EB3
 P 6500 2300
-F 0 "#PWR?" H 6500 2150 50  0001 C CNN
+F 0 "#PWR024" H 6500 2150 50  0001 C CNN
 F 1 "+3V3" H 6500 2440 50  0000 C CNN
 F 2 "" H 6500 2300 50  0001 C CNN
@@
 $EndComp
 $Comp
-L +3V3 #PWR?
+L +3V3 #PWR025
 U 1 1 5A9B4ED1
 P 6650 3600
-F 0 "#PWR?" H 6650 3450 50  0001 C CNN
+F 0 "#PWR025" H 6650 3450 50  0001 C CNN
 F 1 "+3V3" H 6650 3740 50  0000 C CNN
 F 2 "" H 6650 3600 50  0001 C CNN
@@
 $EndComp
 $Comp
-L GND #PWR?
+L GND #PWR026
 U 1 1 5A9B4EEF
 P 6500 2600
-F 0 "#PWR?" H 6500 2350 50  0001 C CNN
+F 0 "#PWR026" H 6500 2350 50  0001 C CNN
 F 1 "GND" H 6500 2450 50  0000 C CNN
 F 2 "" H 6500 2600 50  0001 C CNN
@@
 $EndComp
 $Comp
-L GND #PWR?
+L GND #PWR027
 U 1 1 5A9B4F0D
 P 6650 3900
-F 0 "#PWR?" H 6650 3650 50  0001 C CNN
+F 0 "#PWR027" H 6650 3650 50  0001 C CNN
 F 1 "GND" H 6650 3750 50  0000 C CNN
 F 2 "" H 6650 3900 50  0001 C CNN
@@
 	6500 3900 6650 3900
 $Comp
-L Crystal Y?
+L Crystal Y2
 U 1 1 5A9B5181
 P 1800 2850
-F 0 "Y?" H 1800 3000 50  0000 C CNN
+F 0 "Y2" H 1800 3000 50  0000 C CNN
 F 1 "8MHz" H 1800 2700 50  0000 C CNN
 F 2 "" H 1800 2850 50  0001 C CNN
@@
 $EndComp
 $Comp
-L C C?
+L C C9
 U 1 1 5A9B523D
 P 1450 3000
-F 0 "C?" H 1475 3100 50  0000 L CNN
+F 0 "C9" H 1475 3100 50  0000 L CNN
 F 1 "20pF" H 1475 2900 50  0000 L CNN
 F 2 "" H 1488 2850 50  0001 C CNN
@@
 $EndComp
 $Comp
-L C C?
+L C C8
 U 1 1 5A9B5273
 P 1450 2700
-F 0 "C?" H 1475 2800 50  0000 L CNN
+F 0 "C8" H 1475 2800 50  0000 L CNN
 F 1 "20pF" H 1475 2600 50  0000 L CNN
 F 2 "" H 1488 2550 50  0001 C CNN
@@
 $EndComp
 $Comp
-L GND #PWR?
+L GND #PWR028
 U 1 1 5A9B52D9
 P 1100 2850
-F 0 "#PWR?" H 1100 2600 50  0001 C CNN
+F 0 "#PWR028" H 1100 2600 50  0001 C CNN
 F 1 "GND" H 1100 2700 50  0000 C CNN
 F 2 "" H 1100 2850 50  0001 C CNN
@@
 Connection ~ 1300 2850
 $Comp
-L STM32F103CBT6 U?
+L STM32F103CBT6 U4
 U 1 1 5A9B43F1
 P 2500 2500
-F 0 "U?" H 4200 2900 60  0000 C CNN
+F 0 "U4" H 4200 2900 60  0000 C CNN
 F 1 "STM32F103CBT6" H 4200 2800 60  0000 C CNN
 F 2 "LQFP-48" H 4200 2740 60  0001 C CNN
@@
 $EndComp
 $Comp
-L R R?
+L R R14
 U 1 1 5A9E117E
 P 2050 3000
-F 0 "R?" V 2130 3000 50  0000 C CNN
+F 0 "R14" V 2130 3000 50  0000 C CNN
 F 1 "390" V 2050 3000 50  0000 C CNN
 F 2 "" V 1980 3000 50  0001 C CNN
@@
 Connection ~ 1800 2700
 $Comp
-L R R?
+L R R15
 U 1 1 5A9E13C9
 P 6450 2900
-F 0 "R?" V 6530 2900 50  0000 C CNN
+F 0 "R15" V 6530 2900 50  0000 C CNN
 F 1 "10k" V 6450 2900 50  0000 C CNN
 F 2 "" V 6380 2900 50  0001 C CNN
@@
 	6300 2900 5900 2900
 $Comp
-L SW_DPDT_x2 SW?
+L SW_DPDT_x2 SW4
 U 1 1 5A9E145C
 P 6800 2900
-F 0 "SW?" H 6800 3070 50  0000 C CNN
+F 0 "SW4" H 6800 3070 50  0000 C CNN
 F 1 "SW_DPDT_x2" H 6800 2700 50  0000 C CNN
 F 2 "" H 6800 2900 50  0001 C CNN
@@
 $EndComp
 $Comp
-L +3V3 #PWR?
+L +3V3 #PWR029
 U 1 1 5A9E14BA
 P 7150 2800
-F 0 "#PWR?" H 7150 2650 50  0001 C CNN
+F 0 "#PWR029" H 7150 2650 50  0001 C CNN
 F 1 "+3V3" H 7150 2940 50  0000 C CNN
 F 2 "" H 7150 2800 50  0001 C CNN
@@
 $EndComp
 $Comp
-L GND #PWR?
+L GND #PWR030
 U 1 1 5A9E14E4
 P 7150 3000
-F 0 "#PWR?" H 7150 2750 50  0001 C CNN
+F 0 "#PWR030" H 7150 2750 50  0001 C CNN
 F 1 "GND" H 7150 2850 50  0000 C CNN
 F 2 "" H 7150 3000 50  0001 C CNN
@@
 	2150 3300 2500 3300
 $Comp
-L SW_DIP_x01 SW?
+L SW_DIP_x01 SW3
 U 1 1 5A9E1C79
 P 1250 1600
-F 0 "SW?" H 1250 1750 50  0000 C CNN
+F 0 "SW3" H 1250 1750 50  0000 C CNN
 F 1 "SW_DIP_x01" H 1250 1450 50  0000 C CNN
 F 2 "" H 1250 1600 50  0001 C CNN
@@
 $EndComp
 $Comp
-L C C?
+L C C5
 U 1 1 5A9E1D22
 P 1250 1950
-F 0 "C?" H 1275 2050 50  0000 L CNN
+F 0 "C5" H 1275 2050 50  0000 L CNN
 F 1 "100nF" H 1275 1850 50  0000 L CNN
 F 2 "" H 1288 1800 50  0001 C CNN
@@
 	950  1950 950  1600
 $Comp
-L GND #PWR?
+L GND #PWR031
 U 1 1 5A9E1E52
 P 950 1950
-F 0 "#PWR?" H 950 1700 50  0001 C CNN
+F 0 "#PWR031" H 950 1700 50  0001 C CNN
 F 1 "GND" H 950 1800 50  0000 C CNN
 F 2 "" H 950 1950 50  0001 C CNN
@@
 RESET
 $Comp
-L Crystal Y?
+L Crystal Y1
 U 1 1 5A9E338A
 P 1800 2350
-F 0 "Y?" H 1800 2500 50  0000 C CNN
+F 0 "Y1" H 1800 2500 50  0000 C CNN
 F 1 "32.768kHz" H 1800 2200 50  0000 C CNN
 F 2 "" H 1800 2350 50  0001 C CNN
@@
 $EndComp
 $Comp
-L C C?
+L C C7
 U 1 1 5A9E3390
 P 1450 2500
-F 0 "C?" H 1475 2600 50  0000 L CNN
+F 0 "C7" H 1475 2600 50  0000 L CNN
 F 1 "10pF" H 1475 2400 50  0000 L CNN
 F 2 "" H 1488 2350 50  0001 C CNN
@@
 $EndComp
 $Comp
-L C C?
+L C C6
 U 1 1 5A9E3396
 P 1450 2200
-F 0 "C?" H 1475 2300 50  0000 L CNN
+F 0 "C6" H 1475 2300 50  0000 L CNN
 F 1 "10pF" H 1475 2100 50  0000 L CNN
 F 2 "" H 1488 2050 50  0001 C CNN
@@
 $EndComp
 $Comp
-L GND #PWR?
+L GND #PWR032
 U 1 1 5A9E339C
 P 1100 2350
-F 0 "#PWR?" H 1100 2100 50  0001 C CNN
+F 0 "#PWR032" H 1100 2100 50  0001 C CNN
 F 1 "GND" H 1100 2200 50  0000 C CNN
 F 2 "" H 1100 2350 50  0001 C CNN
@@
 Connection ~ 1300 2350
 $Comp
-L R R?
+L R R13
 U 1 1 5A9E33A5
 P 2050 2500
-F 0 "R?" V 2130 2500 50  0000 C CNN
+F 0 "R13" V 2130 2500 50  0000 C CNN
 F 1 "0" V 2050 2500 50  0000 C CNN
 F 2 "" V 1980 2500 50  0001 C CNN
@@
 	2250 2700 2250 2200
 $Comp
-L Conn_ARM_JTAG_SWD_20 J?
+L Conn_ARM_JTAG_SWD_20 J1
 U 1 1 5A9E398F
 P 8700 3000
-F 0 "J?" H 8500 3850 50  0000 R CNN
+F 0 "J1" H 8500 3850 50  0000 R CNN
 F 1 "Conn_ARM_JTAG_SWD_20" H 8500 3750 50  0000 R BNN
 F 2 "" H 9150 1950 50  0001 L TNN
@@
 $EndComp
 $Comp
-L GND #PWR?
+L GND #PWR033
 U 1 1 5A9E3BB2
 P 8600 3800
-F 0 "#PWR?" H 8600 3550 50  0001 C CNN
+F 0 "#PWR033" H 8600 3550 50  0001 C CNN
 F 1 "GND" H 8600 3650 50  0000 C CNN
 F 2 "" H 8600 3800 50  0001 C CNN
@@
 $EndComp
 $Comp
-L +3V3 #PWR?
+L +3V3 #PWR034
 U 1 1 5A9E3C56
 P 8600 2200
-F 0 "#PWR?" H 8600 2050 50  0001 C CNN
+F 0 "#PWR034" H 8600 2050 50  0001 C CNN
 F 1 "+3V3" H 8600 2340 50  0000 C CNN
 F 2 "" H 8600 2200 50  0001 C CNN
@@
 TCK/SWCLK
 $Comp
-L R R?
+L R R18
 U 1 1 5A9E4E8F
 P 10250 2800
-F 0 "R?" V 10330 2800 50  0000 C CNN
+F 0 "R18" V 10330 2800 50  0000 C CNN
 F 1 "10k" V 10250 2800 50  0000 C CNN
 F 2 "" V 10180 2800 50  0001 C CNN
@@
 $EndComp
 $Comp
-L R R?
+L R R16
 U 1 1 5A9E4F21
 P 9700 3400
-F 0 "R?" V 9780 3400 50  0000 C CNN
+F 0 "R16" V 9780 3400 50  0000 C CNN
 F 1 "10k" V 9700 3400 50  0000 C CNN
 F 2 "" V 9630 3400 50  0001 C CNN
@@
 $EndComp
 $Comp
-L R R?
+L R R17
 U 1 1 5A9E4F7B
 P 9700 3600
-F 0 "R?" V 9780 3600 50  0000 C CNN
+F 0 "R17" V 9780 3600 50  0000 C CNN
 F 1 "10k" V 9700 3600 50  0000 C CNN
 F 2 "" V 9630 3600 50  0001 C CNN
@@
 $EndComp
 $Comp
-L GND #PWR?
+L GND #PWR035
 U 1 1 5A9E4FC5
 P 9850 3700
-F 0 "#PWR?" H 9850 3450 50  0001 C CNN
+F 0 "#PWR035" H 9850 3450 50  0001 C CNN
 F 1 "GND" H 9850 3550 50  0000 C CNN
 F 2 "" H 9850 3700 50  0001 C CNN
@@
 	9300 3400 9550 3400
 $Comp
-L GND #PWR?
+L GND #PWR036
 U 1 1 5A9E51B1
 P 10550 2800
-F 0 "#PWR?" H 10550 2550 50  0001 C CNN
+F 0 "#PWR036" H 10550 2550 50  0001 C CNN
 F 1 "GND" H 10550 2650 50  0000 C CNN
 F 2 "" H 10550 2800 50  0001 C CNN

Commit message: Finished Schematic
Parts:
- removed U4: STM32F103CBT6, LQFP-48, symbol STM32F103CBT6
- added U?: STM32F303CCT6, LQFP-48, symbol STM32F303CCT6
Connections:
- net +3V3: now also U?.1 (VBAT), U?.24 (VDD_1), U?.36 (VDD_2), U?.48 (VDD_3), U?.9 (VDDA)
- net GND: now also U?.23 (VSS_1), U?.35 (VSS_2), U?.47 (VSS_3), U?.8 (VSSA)
- net PA0: now also U?.10 (PA0-WKUP)
- net PA1: now also U?.11 (PA1)
- net PA10: now also U?.31 (PA10)
- net PA11: now also U?.32 (PA11)
- net PA12: now also U?.33 (PA12)
- net PA2: now also U?.12 (PA2)
- net PA3: now also U?.13 (PA3)
- net PA4: now also U?.14 (PA4)
- net PA5: now also U?.15 (PA5)
- net PA6: now also U?.16 (PA6)
- net PA7: now also U?.17 (PA7)
- net PA8: now also U?.29 (PA8)
- net PA9: now also U?.30 (PA9)
- net PB0: now also U?.18 (PB0)
- net PB1: now also U?.19 (PB1)
- net PB10: now also U?.21 (PB10)
- net PB11: now also U?.22 (PB11)
- net PB12: now also U?.25 (PB12)
- net PB13: now also U?.26 (PB13)
- net PB14: now also U?.27 (PB14)
- net PB15: now also U?.28 (PB15)
- net PB2: now also U?.20 (PB2)
- net PB5: now also U?.41 (PB5)
- net PB6: now also U?.42 (PB6)
- net PB7: now also U?.43 (PB7)
- net PB8: now also U?.45 (PB8)
- net PB9: now also U?.46 (PB9)
- net PC13: now also U?.2 (PC13-TAMPER-RTC)
- net RESET: now also U?.7 (NRST)
- net TCK/SWCLK: now also U?.37 (PA14)
- net TDI: now also U?.38 (PA15)
- net TDO/SWO: now also U?.39 (PB3)
- net TMS/SWDIO: now also U?.34 (PA13)
- net TRST: now also U?.40 (PB4)
- net at C6.1, Y1.1: now also U?.3 (PC14-OSC32_IN)
- net at R13.1: now also U?.4 (PC15-OSC32_OUT)
- net at R15.2: now also U?.44 (BOOT0)
- net at C8.1, Y2.1: now also U?.5 (PD0-OSC_IN)
- net at R14.1: now also U?.6 (PD1-OSC_OUT)
Changed lines of the file:
@@
 Connection ~ 1300 2850
-$Comp
-L STM32F103CBT6 U4
-U 1 1 5A9B43F1
-P 2500 2500
-F 0 "U4" H 4200 2900 60  0000 C CNN
-F 1 "STM32F103CBT6" H 4200 2800 60  0000 C CNN
-F 2 "LQFP-48" H 4200 2740 60  0001 C CNN
-F 3 "" H 2500 2500 60  0000 C CNN
-	1    2500 2500
-	1    0    0    -1
-$EndComp
 $Comp
 L R R14
@@
 Text HLabel 2500 2600 0    60   Input ~ 0
 PC13
+$Comp
+L STM32F303CCT6 U?
+U 1 1 5AC15889
+P 2500 2500
+F 0 "U?" H 4200 2900 60  0000 C CNN
+F 1 "STM32F303CCT6" H 4200 2800 60  0000 C CNN
+F 2 "LQFP-48" H 4200 2740 60  0001 C CNN
+F 3 "" H 2500 2500 60  0000 C CNN
+	1    2500 2500
+	1    0    0    -1
+$EndComp
 $EndSCHEMATC
