File: TouchSensing.sch (KiCad schematic (older format))
At the start: 0 parts

Commit message: Added power, touch, and motor controller
Parts:
- added R? (x4): 10k, symbol R
- added SW? (x2): SW_SPDT, symbol SW_SPDT
Connections:
- new net +3V3: SW?.2 (B), SW?.2 (B)
- new net GND: R?.1, R?.1, R?.2, R?.2
- new net T_BackLeft: R?.1, SW?.3 (C)
- new net T_BackRight: R?.1, SW?.3 (C)
- new net T_FrontLeft: R?.2, SW?.1 (A)
- new net T_FrontRight: R?.2, SW?.1 (A)
Changed lines of the file:
@@
 $Descr A4 11693 8268
 encoding utf-8
-Sheet 1 8
+Sheet 4 7
 Title ""
 Date ""
@@
 Comment4 ""
 $EndDescr
+$Comp
+L SW_SPDT SW?
+U 1 1 5AA4E63F
+P 5150 3475
+F 0 "SW?" H 5150 3645 50  0000 C CNN
+F 1 "SW_SPDT" H 5150 3275 50  0000 C CNN
+F 2 "" H 5150 3475 50  0001 C CNN
+F 3 "" H 5150 3475 50  0001 C CNN
+	1    5150 3475
+	1    0    0    -1
+$EndComp
+$Comp
+L R R?
+U 1 1 5AA4E68A
+P 5575 3225
+F 0 "R?" V 5655 3225 50  0000 C CNN
+F 1 "10k" V 5575 3225 50  0000 C CNN
+F 2 "" V 5505 3225 50  0001 C CNN
+F 3 "" H 5575 3225 50  0001 C CNN
+	1    5575 3225
+	1    0    0    -1
+$EndComp
+$Comp
+L R R?
+U 1 1 5AA4E6DF
+P 5575 3725
+F 0 "R?" V 5655 3725 50  0000 C CNN
+F 1 "10k" V 5575 3725 50  0000 C CNN
+F 2 "" V 5505 3725 50  0001 C CNN
+F 3 "" H 5575 3725 50  0001 C CNN
+	1    5575 3725
+	1    0    0    -1
+$EndComp
+$Comp
+L +3V3 #PWR?
+U 1 1 5AA4E728
+P 4950 3475
+F 0 "#PWR?" H 4950 3325 50  0001 C CNN
+F 1 "+3V3" H 4950 3615 50  0000 C CNN
+F 2 "" H 4950 3475 50  0001 C CNN
+F 3 "" H 4950 3475 50  0001 C CNN
+	1    4950 3475
+	1    0    0    -1
+$EndComp
+$Comp
+L GND #PWR?
+U 1 1 5AA4E746
+P 5425 3075
+F 0 "#PWR?" H 5425 2825 50  0001 C CNN
+F 1 "GND" H 5425 2925 50  0000 C CNN
+F 2 "" H 5425 3075 50  0001 C CNN
+F 3 "" H 5425 3075 50  0001 C CNN
+	1    5425 3075
+	1    0    0    -1
+$EndComp
+$Comp
+L GND #PWR?
+U 1 1 5AA4E760
+P 5425 3875
+F 0 "#PWR?" H 5425 3625 50  0001 C CNN
+F 1 "GND" H 5425 3725 50  0000 C CNN
+F 2 "" H 5425 3875 50  0001 C CNN
+F 3 "" H 5425 3875 50  0001 C CNN
+	1    5425 3875
+	1    0    0    -1
+$EndComp
+Wire Wire Line
+	5575 3875 5425 3875
+Wire Wire Line
+	5575 3075 5425 3075
+Wire Wire Line
+	5350 3375 5725 3375
+Wire Wire Line
+	5350 3575 5725 3575
+Text GLabel 5725 3375 2    60   Input ~ 0
+T_FrontLeft
+Connection ~ 5575 3375
+Text GLabel 5725 3575 2    60   Input ~ 0
+T_BackLeft
+Connection ~ 5575 3575
+$Comp
+L SW_SPDT SW?
+U 1 1 5AA4E865
+P 6925 3425
+F 0 "SW?" H 6925 3595 50  0000 C CNN
+F 1 "SW_SPDT" H 6925 3225 50  0000 C CNN
+F 2 "" H 6925 3425 50  0001 C CNN
+F 3 "" H 6925 3425 50  0001 C CNN
+	1    6925 3425
+	1    0    0    -1
+$EndComp
+$Comp
+L R R?
+U 1 1 5AA4E86B
+P 7350 3175
+F 0 "R?" V 7430 3175 50  0000 C CNN
+F 1 "10k" V 7350 3175 50  0000 C CNN
+F 2 "" V 7280 3175 50  0001 C CNN
+F 3 "" H 7350 3175 50  0001 C CNN
+	1    7350 3175
+	1    0    0    -1
+$EndComp
+$Comp
+L R R?
+U 1 1 5AA4E871
+P 7350 3675
+F 0 "R?" V 7430 3675 50  0000 C CNN
+F 1 "10k" V 7350 3675 50  0000 C CNN
+F 2 "" V 7280 3675 50  0001 C CNN
+F 3 "" H 7350 3675 50  0001 C CNN
+	1    7350 3675
+	1    0    0    -1
+$EndComp
+$Comp
+L +3V3 #PWR?
+U 1 1 5AA4E877
+P 6725 3425
+F 0 "#PWR?" H 6725 3275 50  0001 C CNN
+F 1 "+3V3" H 6725 3565 50  0000 C CNN
+F 2 "" H 6725 3425 50  0001 C CNN
+F 3 "" H 6725 3425 50  0001 C CNN
+	1    6725 3425
+	1    0    0    -1
+$EndComp
+$Comp
+L GND #PWR?
+U 1 1 5AA4E87D
+P 7200 3025
+F 0 "#PWR?" H 7200 2775 50  0001 C CNN
+F 1 "GND" H 7200 2875 50  0000 C CNN
+F 2 "" H 7200 3025 50  0001 C CNN
+F 3 "" H 7200 3025 50  0001 C CNN
+	1    7200 3025
+	1    0    0    -1
+$EndComp
+$Comp
+L GND #PWR?
+U 1 1 5AA4E883
+P 7200 3825
+F 0 "#PWR?" H 7200 3575 50  0001 C CNN
+F 1 "GND" H 7200 3675 50  0000 C CNN
+F 2 "" H 7200 3825 50  0001 C CNN
+F 3 "" H 7200 3825 50  0001 C CNN
+	1    7200 3825
+	1    0    0    -1
+$EndComp
+Wire Wire Line
+	7350 3825 7200 3825
+Wire Wire Line
+	7350 3025 7200 3025
+Wire Wire Line
+	7125 3325 7500 3325
+Wire Wire Line
+	7125 3525 7500 3525
+Text GLabel 7500 3325 2    60   Input ~ 0
+T_FrontRight
+Connection ~ 7350 3325
+Text GLabel 7500 3525 2    60   Input ~ 0
+T_BackRight
+Connection ~ 7350 3525
 $EndSCHEMATC

Commit message: Adding IR Sensor
Parts:
- gave numbers to parts that had none: 6
Changed lines of the file:
@@
 $EndDescr
 $Comp
-L SW_SPDT SW?
+L SW_SPDT SW1
 U 1 1 5AA4E63F
 P 5150 3475
-F 0 "SW?" H 5150 3645 50  0000 C CNN
+F 0 "SW1" H 5150 3645 50  0000 C CNN
 F 1 "SW_SPDT" H 5150 3275 50  0000 C CNN
 F 2 "" H 5150 3475 50  0001 C CNN
@@
 $EndComp
 $Comp
-L R R?
+L R R7
 U 1 1 5AA4E68A
 P 5575 3225
-F 0 "R?" V 5655 3225 50  0000 C CNN
+F 0 "R7" V 5655 3225 50  0000 C CNN
 F 1 "10k" V 5575 3225 50  0000 C CNN
 F 2 "" V 5505 3225 50  0001 C CNN
@@
 $EndComp
 $Comp
-L R R?
+L R R8
 U 1 1 5AA4E6DF
 P 5575 3725
-F 0 "R?" V 5655 3725 50  0000 C CNN
+F 0 "R8" V 5655 3725 50  0000 C CNN
 F 1 "10k" V 5575 3725 50  0000 C CNN
 F 2 "" V 5505 3725 50  0001 C CNN
@@
 $EndComp
 $Comp
-L +3V3 #PWR?
+L +3V3 #PWR011
 U 1 1 5AA4E728
 P 4950 3475
-F 0 "#PWR?" H 4950 3325 50  0001 C CNN
+F 0 "#PWR011" H 4950 3325 50  0001 C CNN
 F 1 "+3V3" H 4950 3615 50  0000 C CNN
 F 2 "" H 4950 3475 50  0001 C CNN
@@
 $EndComp
 $Comp
-L GND #PWR?
+L GND #PWR012
 U 1 1 5AA4E746
 P 5425 3075
-F 0 "#PWR?" H 5425 2825 50  0001 C CNN
+F 0 "#PWR012" H 5425 2825 50  0001 C CNN
 F 1 "GND" H 5425 2925 50  0000 C CNN
 F 2 "" H 5425 3075 50  0001 C CNN
@@
 $EndComp
 $Comp
-L GND #PWR?
+L GND #PWR013
 U 1 1 5AA4E760
 P 5425 3875
-F 0 "#PWR?" H 5425 3625 50  0001 C CNN
+F 0 "#PWR013" H 5425 3625 50  0001 C CNN
 F 1 "GND" H 5425 3725 50  0000 C CNN
 F 2 "" H 5425 3875 50  0001 C CNN
@@
 Connection ~ 5575 3575
 $Comp
-L SW_SPDT SW?
+L SW_SPDT SW2
 U 1 1 5AA4E865
 P 6925 3425
-F 0 "SW?" H 6925 3595 50  0000 C CNN
+F 0 "SW2" H 6925 3595 50  0000 C CNN
 F 1 "SW_SPDT" H 6925 3225 50  0000 C CNN
 F 2 "" H 6925 3425 50  0001 C CNN
@@
 $EndComp
 $Comp
-L R R?
+L R R9
 U 1 1 5AA4E86B
 P 7350 3175
-F 0 "R?" V 7430 3175 50  0000 C CNN
+F 0 "R9" V 7430 3175 50  0000 C CNN
 F 1 "10k" V 7350 3175 50  0000 C CNN
 F 2 "" V 7280 3175 50  0001 C CNN
@@
 $EndComp
 $Comp
-L R R?
+L R R10
 U 1 1 5AA4E871
 P 7350 3675
-F 0 "R?" V 7430 3675 50  0000 C CNN
+F 0 "R10" V 7430 3675 50  0000 C CNN
 F 1 "10k" V 7350 3675 50  0000 C CNN
 F 2 "" V 7280 3675 50  0001 C CNN
@@
 $EndComp
 $Comp
-L +3V3 #PWR?
+L +3V3 #PWR014
 U 1 1 5AA4E877
 P 6725 3425
-F 0 "#PWR?" H 6725 3275 50  0001 C CNN
+F 0 "#PWR014" H 6725 3275 50  0001 C CNN
 F 1 "+3V3" H 6725 3565 50  0000 C CNN
 F 2 "" H 6725 3425 50  0001 C CNN
@@
 $EndComp
 $Comp
-L GND #PWR?
+L GND #PWR015
 U 1 1 5AA4E87D
 P 7200 3025
-F 0 "#PWR?" H 7200 2775 50  0001 C CNN
+F 0 "#PWR015" H 7200 2775 50  0001 C CNN
 F 1 "GND" H 7200 2875 50  0000 C CNN
 F 2 "" H 7200 3025 50  0001 C CNN
@@
 $EndComp
 $Comp
-L GND #PWR?
+L GND #PWR016
 U 1 1 5AA4E883
 P 7200 3825
-F 0 "#PWR?" H 7200 3575 50  0001 C CNN
+F 0 "#PWR016" H 7200 3575 50  0001 C CNN
 F 1 "GND" H 7200 3675 50  0000 C CNN
 F 2 "" H 7200 3825 50  0001 C CNN

Commit message: Finished Schematic
Changed lines of the file:
@@
 Wire Wire Line
 	5350 3575 5725 3575
-Text GLabel 5725 3375 2    60   Input ~ 0
-T_FrontLeft
 Connection ~ 5575 3375
-Text GLabel 5725 3575 2    60   Input ~ 0
-T_BackLeft
 Connection ~ 5575 3575
 $Comp
@@
 Wire Wire Line
 	7125 3525 7500 3525
-Text GLabel 7500 3325 2    60   Input ~ 0
+Connection ~ 7350 3325
+Connection ~ 7350 3525
+Text HLabel 5725 3375 2    60   Input ~ 0
+T_FrontLeft
+Text HLabel 5725 3575 2    60   Input ~ 0
+T_BackLeft
+Text HLabel 7500 3325 2    60   Input ~ 0
 T_FrontRight
-Connection ~ 7350 3325
-Text GLabel 7500 3525 2    60   Input ~ 0
+Text HLabel 7500 3525 2    60   Input ~ 0
 T_BackRight
-Connection ~ 7350 3525
 $EndSCHEMATC
