File: _saved_TouchSensing.sch (KiCad schematic (older format))
At the start: 10 parts, among them SW401 SW_SPDT, SW402 SW_SPDT

Commit message: Started associating footprints
Parts:
- R401, R402, R403, R404: footprint (none) -> Resistors_SMD:R_0402
Changed lines of the file:
@@
 F 0 "R401" V 5655 3225 50  0000 C CNN
 F 1 "200" V 5575 3225 50  0000 C CNN
-F 2 "" V 5505 3225 50  0001 C CNN
+F 2 "Resistors_SMD:R_0402" V 5505 3225 50  0001 C CNN
 F 3 "" H 5575 3225 50  0001 C CNN
 	1    5575 3225
@@
 F 0 "R402" V 5655 3725 50  0000 C CNN
 F 1 "200" V 5575 3725 50  0000 C CNN
-F 2 "" V 5505 3725 50  0001 C CNN
+F 2 "Resistors_SMD:R_0402" V 5505 3725 50  0001 C CNN
 F 3 "" H 5575 3725 50  0001 C CNN
 	1    5575 3725
@@
 $EndComp
 $Comp
-L +3V3 #PWR023
+L +3V3 #PWR23
 U 1 1 5AA4E728
 P 4950 3475
-F 0 "#PWR023" H 4950 3325 50  0001 C CNN
+F 0 "#PWR23" H 4950 3325 50  0001 C CNN
 F 1 "+3V3" H 4950 3615 50  0000 C CNN
 F 2 "" H 4950 3475 50  0001 C CNN
@@
 $EndComp
 $Comp
-L GND #PWR024
+L GND #PWR25
 U 1 1 5AA4E746
 P 5825 2775
-F 0 "#PWR024" H 5825 2525 50  0001 C CNN
+F 0 "#PWR25" H 5825 2525 50  0001 C CNN
 F 1 "GND" H 5825 2625 50  0000 C CNN
 F 2 "" H 5825 2775 50  0001 C CNN
@@
 $EndComp
 $Comp
-L GND #PWR025
+L GND #PWR24
 U 1 1 5AA4E760
 P 5375 4175
-F 0 "#PWR025" H 5375 3925 50  0001 C CNN
+F 0 "#PWR24" H 5375 3925 50  0001 C CNN
 F 1 "GND" H 5375 4025 50  0000 C CNN
 F 2 "" H 5375 4175 50  0001 C CNN
@@
 F 0 "R403" V 7430 3175 50  0000 C CNN
 F 1 "200" V 7350 3175 50  0000 C CNN
-F 2 "" V 7280 3175 50  0001 C CNN
+F 2 "Resistors_SMD:R_0402" V 7280 3175 50  0001 C CNN
 F 3 "" H 7350 3175 50  0001 C CNN
 	1    7350 3175
@@
 F 0 "R404" V 7430 3675 50  0000 C CNN
 F 1 "200" V 7350 3675 50  0000 C CNN
-F 2 "" V 7280 3675 50  0001 C CNN
+F 2 "Resistors_SMD:R_0402" V 7280 3675 50  0001 C CNN
 F 3 "" H 7350 3675 50  0001 C CNN
 	1    7350 3675
@@
 $EndComp
 $Comp
-L +3V3 #PWR026
+L +3V3 #PWR26
 U 1 1 5AA4E877
 P 6725 3425
-F 0 "#PWR026" H 6725 3275 50  0001 C CNN
+F 0 "#PWR26" H 6725 3275 50  0001 C CNN
 F 1 "+3V3" H 6725 3565 50  0000 C CNN
 F 2 "" H 6725 3425 50  0001 C CNN
@@
 	5575 4175 5375 4175
 $Comp
-L GND #PWR027
+L GND #PWR28
 U 1 1 5AC70317
 P 7600 2725
-F 0 "#PWR027" H 7600 2475 50  0001 C CNN
+F 0 "#PWR28" H 7600 2475 50  0001 C CNN
 F 1 "GND" H 7600 2575 50  0000 C CNN
 F 2 "" H 7600 2725 50  0001 C CNN
@@
 	7350 2725 7600 2725
 $Comp
-L GND #PWR028
+L GND #PWR27
 U 1 1 5AC70391
 P 7150 4125
-F 0 "#PWR028" H 7150 3875 50  0001 C CNN
+F 0 "#PWR27" H 7150 3875 50  0001 C CNN
 F 1 "GND" H 7150 3975 50  0000 C CNN
 F 2 "" H 7150 4125 50  0001 C CNN
