File: _saved_smallGroundRobot.sch (KiCad schematic (older format))
At the start: 15 parts, among them J101 Conn_01x03, J102 Conn_01x03, J103 Conn_01x03, J104 Conn_01x03, J105 USB_OTG, Q101 Q_NPN_BEC, Q102 Q_NPN_BEC

Commit message: Started associating footprints
Parts:
- D101, D102: footprint (none) -> LEDs:LED_1206
- D103: footprint (none) -> LEDs:LED_0805
- J101, J102, J103, J104: footprint (none) -> Pin_Headers:Pin_Header_Angled_1x03_Pitch1.27mm
- J105: footprint (none) -> Connectors:USB_Micro-B
- R101, R102, R103, R104, R105: footprint (none) -> Resistors_SMD:R_0402
Changed lines of the file:
@@
 F 0 "D103" H 4450 2800 50  0000 C CNN
 F 1 "LED" H 4450 2600 50  0000 C CNN
-F 2 "" H 4450 2700 50  0001 C CNN
+F 2 "LEDs:LED_0805" H 4450 2700 50  0001 C CNN
 F 3 "" H 4450 2700 50  0001 C CNN
 	1    4450 2700
@@
 F 0 "R103" V 4930 2700 50  0000 C CNN
 F 1 "39" V 4850 2700 50  0000 C CNN
-F 2 "" V 4780 2700 50  0001 C CNN
+F 2 "Resistors_SMD:R_0402" V 4780 2700 50  0001 C CNN
 F 3 "" H 4850 2700 50  0001 C CNN
 	1    4850 2700
@@
 $EndComp
 $Comp
-L GND #PWR01
+L GND #PWR5
 U 1 1 5AC56677
 P 5100 2700
-F 0 "#PWR01" H 5100 2450 50  0001 C CNN
+F 0 "#PWR5" H 5100 2450 50  0001 C CNN
 F 1 "GND" H 5100 2550 50  0000 C CNN
 F 2 "" H 5100 2700 50  0001 C CNN
@@
 F 0 "R101" V 3580 4900 50  0000 C CNN
 F 1 "2" V 3500 4900 50  0000 C CNN
-F 2 "" V 3430 4900 50  0001 C CNN
+F 2 "Resistors_SMD:R_0402" V 3430 4900 50  0001 C CNN
 F 3 "" H 3500 4900 50  0001 C CNN
 	1    3500 4900
@@
 F 0 "D101" H 3500 4700 50  0000 C CNN
 F 1 "LED_Headlight" H 3500 4500 50  0000 C CNN
-F 2 "" H 3500 4600 50  0001 C CNN
+F 2 "LEDs:LED_1206" H 3500 4600 50  0001 C CNN
 F 3 "" H 3500 4600 50  0001 C CNN
 	1    3500 4600
@@
 F 0 "J101" H 2650 5450 50  0000 C CNN
 F 1 "Conn_01x03" H 2650 5050 50  0000 C CNN
-F 2 "" H 2650 5250 50  0001 C CNN
+F 2 "Pin_Headers:Pin_Header_Angled_1x03_Pitch1.27mm" H 2650 5250 50  0001 C CNN
 F 3 "" H 2650 5250 50  0001 C CNN
 	1    2650 5250
@@
 F 0 "J103" H 3000 5450 50  0000 C CNN
 F 1 "Conn_01x03" H 3000 5050 50  0000 C CNN
-F 2 "" H 3000 5250 50  0001 C CNN
+F 2 "Pin_Headers:Pin_Header_Angled_1x03_Pitch1.27mm" H 3000 5250 50  0001 C CNN
 F 3 "" H 3000 5250 50  0001 C CNN
 	1    3000 5250
@@
 GND_L1
 $Comp
-L GND #PWR02
+L GND #PWR2
 U 1 1 5AC21B38
 P 2450 5350
-F 0 "#PWR02" H 2450 5100 50  0001 C CNN
+F 0 "#PWR2" H 2450 5100 50  0001 C CNN
 F 1 "GND" H 2450 5200 50  0000 C CNN
 F 2 "" H 2450 5350 50  0001 C CNN
@@
 F 0 "R102" V 3580 6450 50  0000 C CNN
 F 1 "2" V 3500 6450 50  0000 C CNN
-F 2 "" V 3430 6450 50  0001 C CNN
+F 2 "Resistors_SMD:R_0402" V 3430 6450 50  0001 C CNN
 F 3 "" H 3500 6450 50  0001 C CNN
 	1    3500 6450
@@
 F 0 "D102" H 3500 6250 50  0000 C CNN
 F 1 "LED_Headlight" H 3500 6050 50  0000 C CNN
-F 2 "" H 3500 6150 50  0001 C CNN
+F 2 "LEDs:LED_1206" H 3500 6150 50  0001 C CNN
 F 3 "" H 3500 6150 50  0001 C CNN
 	1    3500 6150
@@
 F 0 "J102" H 2650 7000 50  0000 C CNN
 F 1 "Conn_01x03" H 2650 6600 50  0000 C CNN
-F 2 "" H 2650 6800 50  0001 C CNN
+F 2 "Pin_Headers:Pin_Header_Angled_1x03_Pitch1.27mm" H 2650 6800 50  0001 C CNN
 F 3 "" H 2650 6800 50  0001 C CNN
 	1    2650 6800
@@
 F 0 "J104" H 3000 7000 50  0000 C CNN
 F 1 "Conn_01x03" H 3000 6600 50  0000 C CNN
-F 2 "" H 3000 6800 50  0001 C CNN
+F 2 "Pin_Headers:Pin_Header_Angled_1x03_Pitch1.27mm" H 3000 6800 50  0001 C CNN
 F 3 "" H 3000 6800 50  0001 C CNN
 	1    3000 6800
@@
 GND_L2
 $Comp
-L GND #PWR03
+L GND #PWR4
 U 1 1 5AC2896C
 P 2450 6900
-F 0 "#PWR03" H 2450 6650 50  0001 C CNN
+F 0 "#PWR4" H 2450 6650 50  0001 C CNN
 F 1 "GND" H 2450 6750 50  0000 C CNN
 F 2 "" H 2450 6900 50  0001 C CNN
@@
 F 0 "J105" H 5125 1775 50  0000 L CNN
 F 1 "USB_OTG" H 5125 1675 50  0000 L CNN
-F 2 "" H 5475 1275 50  0001 C CNN
+F 2 "Connectors:USB_Micro-B" H 5475 1275 50  0001 C CNN
 F 3 "" H 5475 1275 50  0001 C CNN
 	1    5325 1325
@@
 USB5V
 $Comp
-L GND #PWR04
+L GND #PWR6
 U 1 1 5AC59382
 P 5325 1725
-F 0 "#PWR04" H 5325 1475 50  0001 C CNN
+F 0 "#PWR6" H 5325 1475 50  0001 C CNN
 F 1 "GND" H 5325 1575 50  0000 C CNN
 F 2 "" H 5325 1725 50  0001 C CNN
@@
 F 0 "R104" V 5700 1325 50  0000 C CNN
 F 1 "22" V 5775 1325 50  0000 C CNN
-F 2 "" V 5705 1325 50  0001 C CNN
+F 2 "Resistors_SMD:R_0402" V 5705 1325 50  0001 C CNN
 F 3 "" H 5775 1325 50  0001 C CNN
 	1    5775 1325
@@
 F 0 "R105" V 5855 1425 50  0000 C CNN
 F 1 "22" V 5775 1425 50  0000 C CNN
-F 2 "" V 5705 1425 50  0001 C CNN
+F 2 "Resistors_SMD:R_0402" V 5705 1425 50  0001 C CNN
 F 3 "" H 5775 1425 50  0001 C CNN
 	1    5775 1425
@@
 $EndComp
 $Comp
-L +3V3 #PWR05
+L +3V3 #PWR1
 U 1 1 5AC7D109
 P 2450 5150
-F 0 "#PWR05" H 2450 5000 50  0001 C CNN
+F 0 "#PWR1" H 2450 5000 50  0001 C CNN
 F 1 "+3V3" H 2450 5290 50  0000 C CNN
 F 2 "" H 2450 5150 50  0001 C CNN
@@
 $EndComp
 $Comp
-L +3V3 #PWR06
+L +3V3 #PWR3
 U 1 1 5AC7D286
 P 2450 6700
-F 0 "#PWR06" H 2450 6550 50  0001 C CNN
+F 0 "#PWR3" H 2450 6550 50  0001 C CNN
 F 1 "+3V3" H 2450 6840 50  0000 C CNN
 F 2 "" H 2450 6700 50  0001 C CNN
@@
 IR_IN
 $Comp
-L +3V3 #PWR07
+L +3V3 #PWR7
 U 1 1 5ACAB9F4
 P 9675 2000
-F 0 "#PWR07" H 9675 1850 50  0001 C CNN
+F 0 "#PWR7" H 9675 1850 50  0001 C CNN
 F 1 "+3V3" H 9675 2140 50  0000 C CNN
 F 2 "" H 9675 2000 50  0001 C CNN
@@
 	9500 2000 9675 2000
 $Comp
-L +1V8 #PWR08
+L +1V8 #PWR8
 U 1 1 5ACABC39
 P 9850 2100
-F 0 "#PWR08" H 9850 1950 50  0001 C CNN
+F 0 "#PWR8" H 9850 1950 50  0001 C CNN
 F 1 "+1V8" H 9850 2240 50  0000 C CNN
 F 2 "" H 9850 2100 50  0001 C CNN
