File: MainBoard/TouchSensing.sch (KiCad schematic (older format))
At the start: 10 parts, among them SW401 SW_SPDT, SW402 SW_SPDT

Commit message: Modified schematic for correct footprint
Parts:
- D401, D402, D403, D404: symbol LED -> smallGroundRobot-rescue:LED
- R401, R402, R403, R404: symbol R -> smallGroundRobot-rescue:R
- SW401, SW402: symbol SW_SPDT -> smallGroundRobot-rescue:SW_SPDT
Changed lines of the file:
@@
-EESchema Schematic File Version 2
-LIBS:smallGroundRobot-rescue
-LIBS:power
-LIBS:device
-LIBS:switches
-LIBS:relays
-LIBS:motors
-LIBS:transistors
-LIBS:conn
-LIBS:linear
-LIBS:regul
-LIBS:74xx
-LIBS:cmos4000
-LIBS:adc-dac
-LIBS:memory
-LIBS:xilinx
-LIBS:microcontrollers
-LIBS:dsp
-LIBS:microchip
-LIBS:analog_switches
-LIBS:motorola
-LIBS:texas
-LIBS:intel
-LIBS:audio
-LIBS:interface
-LIBS:digital-audio
-LIBS:philips
-LIBS:display
-LIBS:cypress
-LIBS:siliconi
-LIBS:opto
-LIBS:atmel
-LIBS:contrib
-LIBS:valves
-LIBS:CustomSymbols
+EESchema Schematic File Version 4
 LIBS:smallGroundRobot-cache
-EELAYER 25 0
+EELAYER 26 0
 EELAYER END
 $Descr A4 11693 8268
@@
 $EndDescr
 $Comp
-L SW_SPDT SW401
+L smallGroundRobot-rescue:SW_SPDT SW401
 U 1 1 5AA4E63F
 P 5150 3475
@@
 $EndComp
 $Comp
-L R R401
+L smallGroundRobot-rescue:R R401
 U 1 1 5AA4E68A
 P 5575 3225
@@
 $EndComp
 $Comp
-L R R402
+L smallGroundRobot-rescue:R R402
 U 1 1 5AA4E6DF
 P 5575 3725
@@
 $EndComp
 $Comp
-L +3V3 #PWR023
+L power:+3V3 #PWR023
 U 1 1 5AA4E728
 P 4950 3475
@@
 $EndComp
 $Comp
-L GND #PWR024
+L power:GND #PWR024
 U 1 1 5AA4E746
 P 5825 2775
@@
 $EndComp
 $Comp
-L GND #PWR025
+L power:GND #PWR025
 U 1 1 5AA4E760
 P 5375 4175
@@
 Connection ~ 5575 3575
 $Comp
-L SW_SPDT SW402
+L smallGroundRobot-rescue:SW_SPDT SW402
 U 1 1 5AA4E865
 P 6925 3425
@@
 $EndComp
 $Comp
-L R R403
+L smallGroundRobot-rescue:R R403
 U 1 1 5AA4E86B
 P 7350 3175
@@
 $EndComp
 $Comp
-L R R404
+L smallGroundRobot-rescue:R R404
 U 1 1 5AA4E871
 P 7350 3675
@@
 $EndComp
 $Comp
-L +3V3 #PWR026
+L power:+3V3 #PWR026
 U 1 1 5AA4E877
 P 6725 3425
@@
 T_BackRight
 $Comp
-L LED D401
+L smallGroundRobot-rescue:LED D401
 U 1 1 5AC6F789
 P 5575 2925
@@
 	5575 2775 5825 2775
 $Comp
-L LED D402
+L smallGroundRobot-rescue:LED D402
 U 1 1 5AC6FAFC
 P 5575 4025
@@
 	5575 4175 5375 4175
 $Comp
-L GND #PWR027
+L power:GND #PWR027
 U 1 1 5AC70317
 P 7600 2725
@@
 $EndComp
 $Comp
-L LED D403
+L smallGroundRobot-rescue:LED D403
 U 1 1 5AC7031D
 P 7350 2875
@@
 	7350 2725 7600 2725
 $Comp
-L GND #PWR028
+L power:GND #PWR028
 U 1 1 5AC70391
 P 7150 4125
@@
 $EndComp
 $Comp
-L LED D404
+L smallGroundRobot-rescue:LED D404
 U 1 1 5AC70397
 P 7350 3975
