File: MainBoard/smallGroundRobot.sch (KiCad schematic (older format))
At the start: 7 parts, among them J101 Conn_01x03, J102 Conn_01x03, J105 USB_OTG

Commit message: Modified schematic for correct footprint
Parts:
- D103: symbol LED -> smallGroundRobot-rescue:LED
- J101, J102: footprint Pin_Headers:Pin_Header_Angled_1x03_Pitch1.27mm -> Pin_Headers:Pin_Header_Angled_1x03_Pitch2.54mm; symbol Conn_01x03 -> smallGroundRobot-rescue:Conn_01x03
- J105: symbol USB_OTG -> smallGroundRobot-rescue:USB_OTG
- R103, R104, R105: symbol R -> smallGroundRobot-rescue:R
Changed lines of the file:
@@
-EESchema Schematic File Version 2
-LIBS:smallGroundRobot-rescue
-LIBS:power
-LIBS:device
-LIBS:switches
-LIBS:relays
-LIBS:motors
-LIBS:transistors
-LIBS:conn
-LIBS:linear
-LIBS:regul
-LIBS:74xx
-LIBS:cmos4000
-LIBS:adc-dac
-LIBS:memory
-LIBS:xilinx
-LIBS:microcontrollers
-LIBS:dsp
-LIBS:microchip
-LIBS:analog_switches
-LIBS:motorola
-LIBS:texas
-LIBS:intel
-LIBS:audio
-LIBS:interface
-LIBS:digital-audio
-LIBS:philips
-LIBS:display
-LIBS:cypress
-LIBS:siliconi
-LIBS:opto
-LIBS:atmel
-LIBS:contrib
-LIBS:valves
-LIBS:CustomSymbols
+EESchema Schematic File Version 4
 LIBS:smallGroundRobot-cache
-EELAYER 25 0
+EELAYER 26 0
 EELAYER END
 $Descr A4 11693 8268
@@
 MC2_IN4
 $Comp
-L LED D103
+L smallGroundRobot-rescue:LED D103
 U 1 1 5AC53F8E
 P 4450 2700
@@
 $EndComp
 $Comp
-L R R103
+L smallGroundRobot-rescue:R R103
 U 1 1 5AC54125
 P 4850 2700
@@
 $EndComp
 $Comp
-L GND #PWR01
+L power:GND #PWR01
 U 1 1 5AC56677
 P 5100 2700
@@
 	4300 2700 3800 2700
 $Comp
-L Conn_01x03 J101
+L smallGroundRobot-rescue:Conn_01x03 J101
 U 1 1 5AC1C60C
 P 2650 5250
 F 0 "J101" H 2650 5450 50  0000 C CNN
 F 1 "Conn_01x03" H 2650 5050 50  0000 C CNN
-F 2 "Pin_Headers:Pin_Header_Angled_1x03_Pitch1.27mm" H 2650 5250 50  0001 C CNN
+F 2 "Pin_Headers:Pin_Header_Angled_1x03_Pitch2.54mm" H 2650 5250 50  0001 C CNN
 F 3 "" H 2650 5250 50  0001 C CNN
 	1    2650 5250
@@
 $EndComp
 $Comp
-L GND #PWR02
+L power:GND #PWR02
 U 1 1 5AC21B38
 P 2450 5350
@@
 L1
 $Comp
-L Conn_01x03 J102
+L smallGroundRobot-rescue:Conn_01x03 J102
 U 1 1 5AC28956
 P 2650 6800
 F 0 "J102" H 2650 7000 50  0000 C CNN
 F 1 "Conn_01x03" H 2650 6600 50  0000 C CNN
-F 2 "Pin_Headers:Pin_Header_Angled_1x03_Pitch1.27mm" H 2650 6800 50  0001 C CNN
+F 2 "Pin_Headers:Pin_Header_Angled_1x03_Pitch2.54mm" H 2650 6800 50  0001 C CNN
 F 3 "" H 2650 6800 50  0001 C CNN
 	1    2650 6800
@@
 $EndComp
 $Comp
-L GND #PWR03
+L power:GND #PWR03
 U 1 1 5AC2896C
 P 2450 6900
@@
 Headlights
 $Comp
-L USB_OTG J105
+L smallGroundRobot-rescue:USB_OTG J105
 U 1 1 5AC50028
 P 5325 1325
@@
 USB5V
 $Comp
-L GND #PWR04
+L power:GND #PWR04
 U 1 1 5AC59382
 P 5325 1725
@@
 $EndComp
 Wire Wire Line
-	5225 1725 5625 1725
+	5225 1725 5325 1725
 Text Label 5925 1325 0    60   ~ 0
 D+
@@
 Connection ~ 5325 1725
 $Comp
-L R R104
+L smallGroundRobot-rescue:R R104
 U 1 1 5AC63839
 P 5775 1325
@@
 $EndComp
 $Comp
-L R R105
+L smallGroundRobot-rescue:R R105
 U 1 1 5AC639CC
 P 5775 1425
@@
 $EndComp
 $Comp
-L +3V3 #PWR05
+L power:+3V3 #PWR05
 U 1 1 5AC7D109
 P 2450 5150
@@
 $EndComp
 $Comp
-L +3V3 #PWR06
+L power:+3V3 #PWR06
 U 1 1 5AC7D286
 P 2450 6700
@@
 IR_IN
 $Comp
-L +3V3 #PWR07
+L power:+3V3 #PWR07
 U 1 1 5ACAB9F4
 P 9675 2000
@@
 	9500 2000 9675 2000
 $Comp
-L +1V8 #PWR08
+L power:+1V8 #PWR08
 U 1 1 5ACABC39
 P 9850 2100
@@
 Wire Wire Line
 	9500 2100 9850 2100
+Wire Wire Line
+	5325 1725 5625 1725
 $EndSCHEMATC
