File: MainBoard/ARM.sch (KiCad schematic (older format))
At the start: 18 parts, among them CON1 AVR-JTAG-10, SW1 SW_SPDT, SW601 SW_DIP_x01, U601 STM32F303CCT6, Y601 32.768kHz, Y602 8MHz

Commit message: Modified design to have working 6V
Parts:
- U601: symbol CustomSymbols:STM32F303CCT6 -> smallGroundRobot-rescue:STM32F303CCT6-CustomSymbols
Changed lines of the file:
@@
 PC13
 $Comp
-L CustomSymbols:STM32F303CCT6 U601
+L smallGroundRobot-rescue:STM32F303CCT6-CustomSymbols U601
 U 1 1 5AC15889
 P 2500 2500
