File: MainBoard/IMU.sch (KiCad schematic (older format))
At the start: 10 parts, among them U201 IMU, U202 Level_Shifter_4Channel

Commit message: Modified schematic for correct footprint
Parts:
- C201: symbol C -> smallGroundRobot-rescue:C
- R201, R202, R203, R204, R205, R206, R207: symbol R -> smallGroundRobot-rescue:R
- U201: symbol IMU -> CustomSymbols:IMU
- U202: symbol Level_Shifter_4Channel-RESCUE-smallGroundRobot -> smallGroundRobot-rescue:Level_Shifter_4Channel-RESCUE-smallGroundRobot
Changed lines of the file:
@@
-EESchema Schematic File Version 2
-LIBS:smallGroundRobot-rescue
-LIBS:power
-LIBS:device
-LIBS:switches
-LIBS:relays
-LIBS:motors
-LIBS:transistors
-LIBS:conn
-LIBS:linear
-LIBS:regul
-LIBS:74xx
-LIBS:cmos4000
-LIBS:adc-dac
-LIBS:memory
-LIBS:xilinx
-LIBS:microcontrollers
-LIBS:dsp
-LIBS:microchip
-LIBS:analog_switches
-LIBS:motorola
-LIBS:texas
-LIBS:intel
-LIBS:audio
-LIBS:interface
-LIBS:digital-audio
-LIBS:philips
-LIBS:display
-LIBS:cypress
-LIBS:siliconi
-LIBS:opto
-LIBS:atmel
-LIBS:contrib
-LIBS:valves
-LIBS:CustomSymbols
+EESchema Schematic File Version 4
 LIBS:smallGroundRobot-cache
-EELAYER 25 0
+EELAYER 26 0
 EELAYER END
 $Descr A4 11693 8268
@@
 $EndDescr
 $Comp
-L IMU U201
+L CustomSymbols:IMU U201
 U 1 1 5A13EED2
 P 4025 3925
@@
 $EndComp
 $Comp
-L R R201
+L smallGroundRobot-rescue:R R201
 U 1 1 5A13EED9
 P 2875 3875
@@
 $EndComp
 $Comp
-L C C201
+L smallGroundRobot-rescue:C C201
 U 1 1 5A13EEE0
 P 4225 4725
@@
 $EndComp
 $Comp
-L GND #PWR09
+L power:GND #PWR09
 U 1 1 5A13EEE7
 P 3825 4875
@@
 $EndComp
 $Comp
-L GND #PWR010
+L power:GND #PWR010
 U 1 1 5A13EEED
 P 5125 4025
@@
 NoConn ~ 3375 3825
 $Comp
-L R R205
+L smallGroundRobot-rescue:R R205
 U 1 1 5A13EF1E
 P 7875 4600
@@
 $EndComp
 $Comp
-L R R204
+L smallGroundRobot-rescue:R R204
 U 1 1 5A13EF25
 P 7625 4600
@@
 $EndComp
 $Comp
-L R R206
+L smallGroundRobot-rescue:R R206
 U 1 1 5A13EF2C
 P 8125 4600
@@
 $EndComp
 $Comp
-L R R207
+L smallGroundRobot-rescue:R R207
 U 1 1 5A13EF33
 P 8325 4600
@@
 	7800 3450 7800 3250
 $Comp
-L GND #PWR011
+L power:GND #PWR011
 U 1 1 5A13EF57
 P 6025 3250
@@
 SCL_1V8
 $Comp
-L R R203
+L smallGroundRobot-rescue:R R203
 U 1 1 5A13EF67
 P 6125 4150
@@
 $EndComp
 $Comp
-L R R202
+L smallGroundRobot-rescue:R R202
 U 1 1 5A13EF6E
 P 5900 4150
@@
 INT2
 $Comp
-L GND #PWR012
+L power:GND #PWR012
 U 1 1 5A04C7D6
 P 7725 4850
@@
 Connection ~ 3825 3125
 $Comp
-L Level_Shifter_4Channel-RESCUE-smallGroundRobot U202
+L smallGroundRobot-rescue:Level_Shifter_4Channel-RESCUE-smallGroundRobot U202
 U 1 1 5AA8177A
 P 6975 3750

Commit message: Modified design to have working 6V
Parts:
- U201: symbol CustomSymbols:IMU -> smallGroundRobot-rescue:IMU-CustomSymbols
Changed lines of the file:
@@
 $EndDescr
 $Comp
-L CustomSymbols:IMU U201
+L smallGroundRobot-rescue:IMU-CustomSymbols U201
 U 1 1 5A13EED2
 P 4025 3925
