File: MainBoard/IRSensing.sch (KiCad schematic (older format))
At the start: 7 parts, among them J505 Conn_01x03, J506 Conn_01x03, J507 Conn_01x03, Q501 Q_NPN_BEC, U504 OPB733TR

Commit message: Modified schematic for correct footprint
Parts:
- J505, J506, J507: footprint Pin_Headers:Pin_Header_Angled_1x03_Pitch1.27mm -> Pin_Headers:Pin_Header_Angled_1x03_Pitch2.54mm; symbol Conn_01x03 -> smallGroundRobot-rescue:Conn_01x03
- Q501: symbol Q_NPN_BEC -> smallGroundRobot-rescue:Q_NPN_BEC
- R507, R508: symbol R -> smallGroundRobot-rescue:R
- U504: symbol OPB733TR -> CustomSymbols:OPB733TR
Changed lines of the file:
@@
-EESchema Schematic File Version 2
-LIBS:smallGroundRobot-rescue
-LIBS:power
-LIBS:device
-LIBS:switches
-LIBS:relays
-LIBS:motors
-LIBS:transistors
-LIBS:conn
-LIBS:linear
-LIBS:regul
-LIBS:74xx
-LIBS:cmos4000
-LIBS:adc-dac
-LIBS:memory
-LIBS:xilinx
-LIBS:microcontrollers
-LIBS:dsp
-LIBS:microchip
-LIBS:analog_switches
-LIBS:motorola
-LIBS:texas
-LIBS:intel
-LIBS:audio
-LIBS:interface
-LIBS:digital-audio
-LIBS:philips
-LIBS:display
-LIBS:cypress
-LIBS:siliconi
-LIBS:opto
-LIBS:atmel
-LIBS:contrib
-LIBS:valves
-LIBS:CustomSymbols
+EESchema Schematic File Version 4
 LIBS:smallGroundRobot-cache
-EELAYER 25 0
+EELAYER 26 0
 EELAYER END
 $Descr A4 11693 8268
@@
 $EndDescr
 $Comp
-L GND #PWR029
+L power:GND #PWR029
 U 1 1 5AA80C23
 P 6600 1800
@@
 Vout_IR_1
 $Comp
-L Conn_01x03 J505
+L smallGroundRobot-rescue:Conn_01x03 J505
 U 1 1 5AC5E221
 P 6375 2100
 F 0 "J505" H 6375 2300 50  0000 C CNN
 F 1 "Conn_01x03" H 6375 1900 50  0000 C CNN
-F 2 "Pin_Headers:Pin_Header_Angled_1x03_Pitch1.27mm" H 6375 2100 50  0001 C CNN
+F 2 "Pin_Headers:Pin_Header_Angled_1x03_Pitch2.54mm" H 6375 2100 50  0001 C CNN
 F 3 "" H 6375 2100 50  0001 C CNN
 	1    6375 2100
@@
 	6175 1800 6600 1800
 $Comp
-L GND #PWR030
+L power:GND #PWR030
 U 1 1 5AC5EDFB
 P 6600 2825
@@
 Vout_IR_2
 $Comp
-L Conn_01x03 J506
+L smallGroundRobot-rescue:Conn_01x03 J506
 U 1 1 5AC5EE16
 P 6375 3125
 F 0 "J506" H 6375 3325 50  0000 C CNN
 F 1 "Conn_01x03" H 6375 2925 50  0000 C CNN
-F 2 "Pin_Headers:Pin_Header_Angled_1x03_Pitch1.27mm" H 6375 3125 50  0001 C CNN
+F 2 "Pin_Headers:Pin_Header_Angled_1x03_Pitch2.54mm" H 6375 3125 50  0001 C CNN
 F 3 "" H 6375 3125 50  0001 C CNN
 	1    6375 3125
@@
 	6175 2825 6600 2825
 $Comp
-L GND #PWR031
+L power:GND #PWR031
 U 1 1 5AC5EFE8
 P 6600 3800
@@
 Vout_IR_3
 $Comp
-L Conn_01x03 J507
+L smallGroundRobot-rescue:Conn_01x03 J507
 U 1 1 5AC5F003
 P 6375 4100
 F 0 "J507" H 6375 4300 50  0000 C CNN
 F 1 "Conn_01x03" H 6375 3900 50  0000 C CNN
-F 2 "Pin_Headers:Pin_Header_Angled_1x03_Pitch1.27mm" H 6375 4100 50  0001 C CNN
+F 2 "Pin_Headers:Pin_Header_Angled_1x03_Pitch2.54mm" H 6375 4100 50  0001 C CNN
 F 3 "" H 6375 4100 50  0001 C CNN
 	1    6375 4100
@@
 	6175 3800 6600 3800
 $Comp
-L OPB733TR U504
+L CustomSymbols:OPB733TR U504
 U 1 1 5AC5F0CD
 P 8500 5200
@@
 	9050 5100 9350 5100
 $Comp
-L R R507
+L smallGroundRobot-rescue:R R507
 U 1 1 5AC5F0D5
 P 7650 5100
@@
 $EndComp
 $Comp
-L R R508
+L smallGroundRobot-rescue:R R508
 U 1 1 5AC5F0DB
 P 7650 5300
@@
 	7250 5100 7500 5100
 $Comp
-L GND #PWR032
+L power:GND #PWR032
 U 1 1 5AC5F0E5
 P 9350 5100
@@
 Main Board
 $Comp
-L Q_NPN_BEC Q501
+L smallGroundRobot-rescue:Q_NPN_BEC Q501
 U 1 1 5AC96FCA
 P 7850 1800
@@
 D_SIG
 $Comp
-L +3V3 #PWR033
+L power:+3V3 #PWR033
 U 1 1 5AC9715B
 P 7950 1600

Commit message: Modified design to have working 6V
Parts:
- U504: symbol CustomSymbols:OPB733TR -> smallGroundRobot-rescue:OPB733TR-CustomSymbols
Changed lines of the file:
@@
 	6175 3800 6600 3800
 $Comp
-L CustomSymbols:OPB733TR U504
+L smallGroundRobot-rescue:OPB733TR-CustomSymbols U504
 U 1 1 5AC5F0CD
 P 8500 5200
