File: MainBoard/MotorController.sch (KiCad schematic (older format))
At the start: 14 parts, among them M301 Motor_DC, M302 Motor_DC, M303 Motor_DC, M304 Motor_DC, U301 A3916, U302 A3916

Commit message: Modified schematic for correct footprint
Parts:
- C301, C303: symbol C -> smallGroundRobot-rescue:C
- M301, M302, M303, M304: symbol Motor_DC -> smallGroundRobot-rescue:Motor_DC
- R301, R302, R303, R304, R305, R306: symbol R -> smallGroundRobot-rescue:R
- U301, U302: footprint Housings_DFN_QFN:DFN-14-1EP_3x3mm_Pitch0.4mm -> Housings_DFN_QFN:QFN-16-1EP_3x3mm_Pitch0.5mm_ThermalVias; symbol A3916 -> CustomSymbols:A3916
Connections:
- no-connect marks 0 -> 2
Changed lines of the file:
@@
-EESchema Schematic File Version 2
-LIBS:smallGroundRobot-rescue
-LIBS:power
-LIBS:device
-LIBS:switches
-LIBS:relays
-LIBS:motors
-LIBS:transistors
-LIBS:conn
-LIBS:linear
-LIBS:regul
-LIBS:74xx
-LIBS:cmos4000
-LIBS:adc-dac
-LIBS:memory
-LIBS:xilinx
-LIBS:microcontrollers
-LIBS:dsp
-LIBS:microchip
-LIBS:analog_switches
-LIBS:motorola
-LIBS:texas
-LIBS:intel
-LIBS:audio
-LIBS:interface
-LIBS:digital-audio
-LIBS:philips
-LIBS:display
-LIBS:cypress
-LIBS:siliconi
-LIBS:opto
-LIBS:atmel
-LIBS:contrib
-LIBS:valves
-LIBS:CustomSymbols
+EESchema Schematic File Version 4
 LIBS:smallGroundRobot-cache
-EELAYER 25 0
+EELAYER 26 0
 EELAYER END
 $Descr A4 11693 8268
@@
 $EndDescr
 $Comp
-L A3916 U301
+L CustomSymbols:A3916 U301
 U 1 1 5AA4F077
 P 3800 3850
 F 0 "U301" H 3800 3750 60  0000 C CNN
 F 1 "A3916" H 3800 3950 60  0000 C CNN
-F 2 "Housings_DFN_QFN:DFN-14-1EP_3x3mm_Pitch0.4mm" H 3800 3850 60  0001 C CNN
+F 2 "Housings_DFN_QFN:QFN-16-1EP_3x3mm_Pitch0.5mm_ThermalVias" H 3800 3850 60  0001 C CNN
 F 3 "" H 3800 3850 60  0001 C CNN
 	1    3800 3850
@@
 MC1_IN4
 $Comp
-L R R301
+L smallGroundRobot-rescue:R R301
 U 1 1 5AA4F12C
 P 2950 4100
@@
 	2500 4100 2800 4100
 $Comp
-L GND #PWR013
+L power:GND #PWR013
 U 1 1 5AA4F189
 P 3100 4200
@@
 $EndComp
 $Comp
-L C C301
+L smallGroundRobot-rescue:C C301
 U 1 1 5AA4F1A9
 P 4700 3450
@@
 Connection ~ 4700 3600
 $Comp
-L Motor_DC M301
+L smallGroundRobot-rescue:Motor_DC M301
 U 1 1 5AA50637
 P 5125 3900
@@
 $EndComp
 $Comp
-L Motor_DC M302
+L smallGroundRobot-rescue:Motor_DC M302
 U 1 1 5AA506D8
 P 5125 4500
@@
 	4925 4200 5125 4200
 $Comp
-L R R303
+L smallGroundRobot-rescue:R R303
 U 1 1 5AA50734
 P 4650 3900
@@
 $EndComp
 $Comp
-L GND #PWR014
+L power:GND #PWR014
 U 1 1 5AA5078D
 P 4800 3900
@@
 	4650 4800 5125 4800
 $Comp
-L R R302
+L smallGroundRobot-rescue:R R302
 U 1 1 5AA507E1
 P 4500 4350
@@
 $EndComp
 $Comp
-L GND #PWR015
+L power:GND #PWR015
 U 1 1 5AA5082F
 P 4500 4500
@@
 $EndComp
 $Comp
-L A3916 U302
+L CustomSymbols:A3916 U302
 U 1 1 5AA50C8A
 P 7600 3850
 F 0 "U302" H 7600 3750 60  0000 C CNN
 F 1 "A3916" H 7600 3950 60  0000 C CNN
-F 2 "Housings_DFN_QFN:DFN-14-1EP_3x3mm_Pitch0.4mm" H 7600 3850 60  0001 C CNN
+F 2 "Housings_DFN_QFN:QFN-16-1EP_3x3mm_Pitch0.5mm_ThermalVias" H 7600 3850 60  0001 C CNN
 F 3 "" H 7600 3850 60  0001 C CNN
 	1    7600 3850
@@
 MC2_IN4
 $Comp
-L R R304
+L smallGroundRobot-rescue:R R304
 U 1 1 5AA50C95
 P 6750 4100
@@
 	6300 4100 6600 4100
 $Comp
-L GND #PWR016
+L power:GND #PWR016
 U 1 1 5AA50CA2
 P 6900 4200
@@
 $EndComp
 $Comp
-L C C303
+L smallGroundRobot-rescue:C C303
 U 1 1 5AA50CA8
 P 8500 3450
@@
 	8300 3600 9100 3600
 $Comp
-L Motor_DC M303
+L smallGroundRobot-rescue:Motor_DC M303
 U 1 1 5AA50CC1
 P 8925 3900
@@
 $EndComp
 $Comp
-L Motor_DC M304
+L smallGroundRobot-rescue:Motor_DC M304
 U 1 1 5AA50CC7
 P 8925 4500
@@
 	8725 4200 8925 4200
 $Comp
-L R R306
+L smallGroundRobot-rescue:R R306
 U 1 1 5AA50CD1
 P 8450 3900
@@
 $EndComp
 $Comp
-L GND #PWR017
+L power:GND #PWR017
 U 1 1 5AA50CD7
 P 8600 3900
@@
 	8450 4800 8925 4800
 $Comp
-L R R305
+L smallGroundRobot-rescue:R R305
 U 1 1 5AA50CE3
 P 8300 4350
@@
 $EndComp
 $Comp
-L GND #PWR018
+L power:GND #PWR018
 U 1 1 5AA50CE9
 P 8300 4500
@@
 $EndComp
 $Comp
-L +3V3 #PWR019
+L power:+3V3 #PWR019
 U 1 1 5AC691BA
 P 2500 4100
@@
 $EndComp
 $Comp
-L +3V3 #PWR020
+L power:+3V3 #PWR020
 U 1 1 5AC693DE
 P 6300 4100
@@
 $EndComp
 $Comp
-L +6V #PWR021
+L power:+6V #PWR021
 U 1 1 5AD38250
 P 9100 3600
@@
 $EndComp
 $Comp
-L +6V #PWR022
+L power:+6V #PWR022
 U 1 1 5AD3873D
 P 5100 3600
@@
 Wire Wire Line
 	4500 3600 5100 3600
+NoConn ~ 3100 3500
+NoConn ~ 6900 3500
 $EndSCHEMATC

Commit message: Modified design to have working 6V
Parts:
- U301, U302: symbol CustomSymbols:A3916 -> smallGroundRobot-rescue:A3916-CustomSymbols
Changed lines of the file:
@@
 $EndDescr
 $Comp
-L CustomSymbols:A3916 U301
+L smallGroundRobot-rescue:A3916-CustomSymbols U301
 U 1 1 5AA4F077
 P 3800 3850
@@
 $EndComp
 $Comp
-L CustomSymbols:A3916 U302
+L smallGroundRobot-rescue:A3916-CustomSymbols U302
 U 1 1 5AA50C8A
 P 7600 3850
