File: MainBoard/Power.sch (KiCad schematic (older format))
At the start: 35 parts, among them J701 Screw_Terminal_01x02, U1 ST8R00WPUR, U701 TPS62237, U702 TPS62231, U703 BQ2423

Commit message: Modified schematic for correct footprint
Parts:
- C1, C701, C702, C703, C704, C705, C706, C707: symbol C -> smallGroundRobot-rescue:C
- D1, D701, D702, D703, D704, D705: symbol LED -> smallGroundRobot-rescue:LED
- J701: symbol Screw_Terminal_01x02 -> smallGroundRobot-rescue:Screw_Terminal_01x02
- L1, L701, L702: symbol L -> smallGroundRobot-rescue:L
- R1: value 10k -> 2.55k; symbol R -> smallGroundRobot-rescue:R
- R2: value 2.55k -> 10k; symbol R -> smallGroundRobot-rescue:R
- R3, R701, R702, R703, R704, R705, R706, R707, R708, R709, R710: symbol R -> smallGroundRobot-rescue:R
- U1: symbol ST8R00WPUR -> CustomSymbols:ST8R00WPUR
- U701, U702: symbol TPS6223x -> CustomSymbols:TPS6223x
- U703: symbol BQ2423 -> CustomSymbols:BQ2423

Commit message: Modified design to have working 6V
Parts:
- U1: symbol CustomSymbols:ST8R00WPUR -> smallGroundRobot-rescue:ST8R00WPUR-CustomSymbols
- U701, U702: symbol CustomSymbols:TPS6223x -> smallGroundRobot-rescue:TPS6223x-CustomSymbols
- U703: symbol CustomSymbols:BQ2423 -> smallGroundRobot-rescue:BQ2423-CustomSymbols
Changed lines of the file:
@@
 $EndComp
 $Comp
-L CustomSymbols:TPS6223x U701
+L smallGroundRobot-rescue:TPS6223x-CustomSymbols U701
 U 1 1 59FB2336
 P 2725 2450
@@
 $EndComp
 $Comp
-L CustomSymbols:BQ2423 U703
+L smallGroundRobot-rescue:BQ2423-CustomSymbols U703
 U 1 1 59FB3951
 P 8525 3650
@@
 $EndComp
 $Comp
-L CustomSymbols:TPS6223x U702
+L smallGroundRobot-rescue:TPS6223x-CustomSymbols U702
 U 1 1 5AC52E2D
 P 2725 4100
@@
 $EndComp
 $Comp
-L CustomSymbols:ST8R00WPUR U1
+L smallGroundRobot-rescue:ST8R00WPUR-CustomSymbols U1
 U 1 1 5AD339E5
 P 2700 6050
